File: hardware/prismatic-spray/ps-daughter/ps-daughter.kicad_pcb (KiCad board)
At the start: 2 copper layers, 85 x 22 mm, 7 parts, among them J1 Conn_01x04_Male

Commit message: PCB Rev 1
Hardware rev 1
- Main board
- Daughter board
Parts:
- removed H1, H2: MountingHole, MountingHole:MountingHole_2.7mm_M2.5
Other:
- outline, holes or cut-outs redrawn
Changed lines of the file:
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@@
   (net 6 "Net-(D3-Pad2)")
   (net 7 "unconnected-(D4-Pad2)")
-  (footprint "MountingHole:MountingHole_2.7mm_M2.5" (layer "F.Cu")
-    (at 38.65 90.55)
-    (descr "Mounting Hole 2.7mm, no annular, M2.5")
-    (tags "mounting hole 2.7mm no annular m2.5")
-    (property "Sheetfile" "ps-daughter.kicad_sch")
-    (property "Sheetname" "")
-    (attr exclude_from_pos_files)
-    (fp_text reference "H1" (at 0 -3.7) (layer "F.SilkS")
-      (effects (font (size 1 1) (thickness 0.15)))
-    )
-    (fp_text value "MountingHole" (at 0 3.7) (layer "F.Fab")
-      (effects (font (size 1 1) (thickness 0.15)))
-    )
-    (fp_text user "${REFERENCE}" (at 0 0) (layer "F.Fab")
-      (effects (font (size 1 1) (thickness 0.15)))
-    )
-    (fp_circle (center 0 0) (end 2.7 0) (layer "Cmts.User") (width 0.15) (fill none))
-    (fp_circle (center 0 0) (end 2.95 0) (layer "F.CrtYd") (width 0.05) (fill none))
-    (pad "" np_thru_hole circle (at 0 0) (size 2.7 2.7) (drill 2.7) (layers *.Cu *.Mask))
-  )
-  (footprint "MountingHole:MountingHole_2.7mm_M2.5" (layer "F.Cu")
-    (at 31.7 90.55)
-    (descr "Mounting Hole 2.7mm, no annular, M2.5")
-    (tags "mounting hole 2.7mm no annular m2.5")
-    (property "Sheetfile" "ps-daughter.kicad_sch")
-    (property "Sheetname" "")
-    (attr exclude_from_pos_files)
-    (fp_text reference "H2" (at 0 -3.7) (layer "F.SilkS")
-      (effects (font (size 1 1) (thickness 0.15)))
-    )
-    (fp_text value "MountingHole" (at 0 3.7) (layer "F.Fab")
-      (effects (font (size 1 1) (thickness 0.15)))
-    )
-    (fp_text user "${REFERENCE}" (at 0 0) (layer "F.Fab")
-      (effects (font (size 1 1) (thickness 0.15)))
-    )
-    (fp_circle (center 0 0) (end 2.7 0) (layer "Cmts.User") (width 0.15) (fill none))
-    (fp_circle (center 0 0) (end 2.95 0) (layer "F.CrtYd") (width 0.05) (fill none))
-    (pad "" np_thru_hole circle (at 0 0) (size 2.7 2.7) (drill 2.7) (layers *.Cu *.Mask))
-  )
   (footprint "LED_SMD:LED_WS2812B_PLCC4_5.0x5.0mm_P3.2mm" (layer "F.Cu")
     (at 107.566666 60.7 90)
@@
   )
   (gr_rect (start 55 55) (end 130 67) (layer "F.SilkS") (width 0.15) (fill none))
-  (gr_rect (start 50 50) (end 135 72) (layer "Edge.Cuts") (width 0.2) (fill none))
+  (gr_line (start 132 72) (end 53 72) (layer "Edge.Cuts") (width 0.2))
+  (gr_arc (start 132 50) (mid 134.12132 50.87868) (end 135 53) (layer "Edge.Cuts") (width 0.2))
+  (gr_arc (start 53 72) (mid 50.87868 71.12132) (end 50 69) (layer "Edge.Cuts") (width 0.2))
+  (gr_line (start 53 50) (end 132 50) (layer "Edge.Cuts") (width 0.2))
+  (gr_line (start 50 53) (end 50 69) (layer "Edge.Cuts") (width 0.2))
+  (gr_arc (start 135 69) (mid 134.12132 71.12132) (end 132 72) (layer "Edge.Cuts") (width 0.2))
+  (gr_arc (start 50 53) (mid 50.87868 50.87868) (end 53 50) (layer "Edge.Cuts") (width 0.2))
+  (gr_line (start 135 53) (end 135 69) (layer "Edge.Cuts") (width 0.2))
   (segment (start 105.966666 63.15) (end 107.041177 64.224511) (width 0.25) (layer "F.Cu") (net 1))
   (segment (start 71.1 63.15) (end 72.174511 64.224511) (width 0.25) (layer "F.Cu") (net 1))
